Commit message: new gazebo

File: rokae/src/gazebo_link_attacher_ws/src/fmauch_universal_robot/ur_description/urdf/battery_pack_sleeve/battery_pack.urdf.xacro (robot description, xacro)
@@ -45,7 +45,4 @@
     </collision>
   </link>
-  <gazebo reference="battery_pack_base_link">
-     <material>Gazebo/Blue</material>
-  </gazebo>
   <link
     name="M6_1_Link">
