Commit message: latest simulation model

File: rokae/src/gazebo_link_attacher_ws/src/battery_pack/urdf/battery_pack.urdf (robot description, URDF)
Before this commit: robot battery_pack, 11 links, 10 joints
Links:
- link M10_2_Link: mass 0.003184 -> 0.00318400891749434
- link M6_2_Link: mass 0.0013212 -> 0.0013211670322828
- link M6_3_Link: mass 0.0013212 -> 0.00132116703228283
- link M8_1_Link: mass 0.0021494 -> 0.00214941637065255
- link M8_2_Link: mass 0.0021494 -> 0.00214941637065243
- link M8_3_Link: mass 0.0021494 -> 0.00214941637065255
- link battery_pack_base_link: mass 590.168232442056 -> 662.17
Joints:
- joint M10_1_Joint: origin xyz=0.2215 -0.196 0.051 rpy=0 0 0 -> xyz=0.521499999999999 -0.195999999999999 0.051 rpy=0 0 0
- joint M10_2_Joint: axis 0 0 1 -> 0 0 0; origin xyz=0.2215 -0.296 0.051 rpy=0 0 0 -> xyz=0.5215 -0.296 0.051 rpy=0 0 0
- joint M10_3_Joint: origin xyz=0.2215 -0.396 0.051 rpy=0 0 0 -> xyz=0.521499999999995 -0.396000000000006 0.051 rpy=0 0 0
- joint M6_1_Joint: origin xyz=0.2215 0.404 0.051 rpy=0 0 0 -> xyz=0.521499999999999 0.404 0.051 rpy=0 0 0
- joint M6_2_Joint: origin xyz=0.2215 0.304 0.051 rpy=0 0 0 -> xyz=0.521499999999999 0.304000000000001 0.051 rpy=0 0 0
- joint M6_3_Joint: origin xyz=0.2215 0.204 0.051 rpy=0 0 0 -> xyz=0.521499999999999 0.204000000000001 0.051 rpy=0 0 0
- joint M8_1_Joint: origin xyz=0.2215 0.104 0.051 rpy=0 0 0 -> xyz=0.521499999999999 0.104000000000001 0.051 rpy=0 0 0
- joint M8_2_Joint: origin xyz=0.2215 0.004 0.051 rpy=0 0 0 -> xyz=0.5215 0.00400000000000017 0.051 rpy=0 0 0
- joint M8_3_Joint: origin xyz=0.2215 -0.096 0.051 rpy=0 0 0 -> xyz=0.521499999999999 -0.0959999999999996 0.051 rpy=0 0 0
- joint sleeve_plate_Joint: axis 0 0 1 -> 0 0 0

File: rokae/src/gazebo_link_attacher_ws/src/fmauch_universal_robot/ur_description/urdf/inc/ur_macro.xacro (robot description, xacro)
@@ -316,679 +316,7 @@
       <child link="${prefix}tool0"/>
     </joint>
-    <link
-    name="endeffector_base_link">
-    <inertial>
-      <origin
-        xyz="-0.0091552 -0.0017971 0.10907"
-        rpy="0 0 0" />
-      <mass
-        value="0.6995" />
-      <inertia
-        ixx="0.00093618"
-        ixy="-1.2386E-06"
-        ixz="-2.4247E-05"
-        iyy="0.0018881"
-        iyz="9.7308E-06"
-        izz="0.0012009" />
-    </inertial>
-    <visual>
-      <origin
-        xyz="0 0 0"
-        rpy="0 0 0" />
-      <geometry>
-        <mesh
-          filename="package://endeffector/meshes/endeffector_base_link.STL" />
-      </geometry>
-      <material
-        name="">
-        <color
-          rgba="0.79216 0.81961 0.93333 1" />
-      </material>
-    </visual>
-    <collision>
-      <origin
-        xyz="0 0 0"
-        rpy="0 0 0" />
-      <geometry>
-        <mesh
-          filename="package://endeffector/meshes/endeffector_base_link.STL" />
-      </geometry>
-    </collision>
-  </link>
-  <link
-    name="camera_Link">
-    <inertial>
-      <origin
-        xyz="-0.013488 -7.0938E-05 -0.013332"
-        rpy="0 0 0" />
-      <mass
-        value="0.071592" />
-      <inertia
-        ixx="2.0232E-05"
-        ixy="-4.6475E-08"
-        ixz="-5.1114E-10"
-        iyy="1.9381E-05"
-        iyz="4.5469E-09"
-        izz="3.1685E-05" />
-    </inertial>
-    <visual>
-      <origin
-        xyz="0 0 0"
-        rpy="0 0 0" />
-      <geometry>
-        <mesh
-          filename="package://endeffector/meshes/camera_Link.STL" />
-      </geometry>
-      <material
-        name="">
-        <color
-          rgba="0.79216 0.81961 0.93333 1" />
-      </material>
-    </visual>
-    <collision>
-      <origin
-        xyz="0 0 0"
-        rpy="0 0 0" />
-      <geometry>
-        <mesh
-          filename="package://endeffector/meshes/camera_Link.STL" />
-      </geometry>
-    </collision>
-  </link>
-  <joint
-    name="camera_Joint"
-    type="fixed">
-    <origin
-      xyz="0.18055 -0.00029745 0.071047"
-      rpy="0.00018844 -0.10472 0" />
-    <parent
-      link="endeffector_base_link" />
-    <child
-      link="camera_Link" />
-    <axis
-      xyz="0 0 0" />
-  </joint>
-    <joint name="${prefix}tool0-endeffector_base_link" type="fixed">
-      <!-- default toolframe: X+ left, Y+ up, Z+ front -->
-      <origin xyz="0 0 0.002" rpy="0 0 ${pi/1.0}"/>
-      <parent link="${prefix}tool0"/>
-      <child link="${prefix}endeffector_base_link"/>
-    </joint>
-<!-- battery_pack -->
-    <link
-      name="battery_pack_base_link">
-      <inertial>
-        <origin
-          xyz="0.840460078869128 0.000748250275173445 -0.0747991952974527"
-          rpy="0 0 0" />
-        <mass
-          value="590.168232442056" />
-        <inertia
-          ixx="68.4216428304914"
-          ixy="0.000761839613148307"
-          ixz="6.32020891220886E-09"
-          iyy="184.407037358386"
-          iyz="1.60985543868867E-09"
-          izz="249.53932694368" />
-      </inertial>
-      <visual>
-        <origin
-          xyz="0 0 0"
-          rpy="0 0 0" />
-        <geometry>
-          <mesh
-            filename="package://battery_pack/meshes/battery_pack_base_link.STL" />
-        </geometry>
-        <material
-          name="">
-          <color
-            rgba="1 1 1 1" />
-        </material>
-      </visual>
-      <collision>
-        <origin
-          xyz="0 0 0"
-          rpy="0 0 0" />
-        <geometry>
-          <mesh
-            filename="package://battery_pack/meshes/battery_pack_base_link.STL" />
-        </geometry>
-      </collision>
-    </link>
-    <link
-      name="M6_1_Link">
-      <inertial>
-        <origin
-          xyz="-1.5781E-08 1.7199E-07 -0.013589"
-          rpy="0 0 0" />
-        <mass
-          value="0.0013212" />
-        <inertia
-          ixx="1.3904E-07"
-          ixy="-5.0602E-13"
-          ixz="5.5231E-11"
-          iyy="1.3904E-07"
-          iyz="-1.7203E-11"
-          izz="1.0587E-08" />
-      </inertial>
-      <visual>
-        <origin
-          xyz="0 0 0"
-          rpy="0 0 0" />
-        <geometry>
-          <mesh
-            filename="package://battery_pack/meshes/M6_1_Link.STL" />
-        </geometry>
-        <material
-          name="">
-          <color
-            rgba="1 1 1 1" />
-        </material>
-      </visual>
-      <collision>
-        <origin
-          xyz="0 0 0"
-          rpy="0 0 0" />
-        <geometry>
-          <mesh
-            filename="package://battery_pack/meshes/M6_1_Link.STL" />
-        </geometry>
-      </collision>
-    </link>
-    <joint
-      name="M6_1_Joint"
-      type="fixed">
-      <origin
-        xyz="0.2215 0.404 0.051"
-        rpy="0 0 0" />
-      <parent
-        link="battery_pack_base_link" />
-      <child
-        link="M6_1_Link" />
-      <axis
-        xyz="0 0 1" />
-    </joint>
-    <link
-      name="M6_2_Link">
-      <inertial>
-        <origin
-          xyz="-1.6918E-07 -3.4772E-08 -0.013589"
-          rpy="0 0 0" />
-        <mass
-          value="0.0013212" />
-        <inertia
-          ixx="1.3904E-07"
-          ixy="7.5348E-13"
-          ixz="1.0967E-11"
-          iyy="1.3904E-07"
-          iyz="5.6799E-11"
-          izz="1.0587E-08" />
-      </inertial>
-      <visual>
-        <origin
-          xyz="0 0 0"
-          rpy="0 0 0" />
-        <geometry>
-          <mesh
-            filename="package://battery_pack/meshes/M6_2_Link.STL" />
-        </geometry>
-        <material
-          name="">
-          <color
-            rgba="1 1 1 1" />
-        </material>
-      </visual>
-      <collision>
-        <origin
-          xyz="0 0 0"
-          rpy="0 0 0" />
-        <geometry>
-          <mesh
-            filename="package://battery_pack/meshes/M6_2_Link.STL" />
-        </geometry>
-      </collision>
-    </link>
-    <joint
-      name="M6_2_Joint"
-      type="fixed">
-      <origin
-        xyz="0.2215 0.304 0.051"
-        rpy="0 0 0" />
-      <parent
-        link="battery_pack_base_link" />
-      <child
-        link="M6_2_Link" />
-      <axis
-        xyz="0 0 1" />
-    </joint>
-    <link
-      name="M6_3_Link">
-      <inertial>
-        <origin
-          xyz="-8.6028E-09 -1.725E-07 -0.013589"
-          rpy="0 0 0" />
-        <mass
-          value="0.0013212" />
-        <inertia
-          ixx="1.3904E-07"
-          ixy="-1.573E-13"
-          ixz="-5.2257E-11"
-          iyy="1.3904E-07"
-          iyz="2.4812E-11"
-          izz="1.0587E-08" />
-      </inertial>
-      <visual>
-        <origin
-          xyz="0 0 0"
-          rpy="0 0 0" />
-        <geometry>
-          <mesh
-            filename="package://battery_pack/meshes/M6_3_Link.STL" />
-        </geometry>
-        <material
-          name="">
-          <color
-            rgba="1 1 1 1" />
-        </material>
-      </visual>
-      <collision>
-        <origin
-          xyz="0 0 0"
-          rpy="0 0 0" />
-        <geometry>
-          <mesh
-            filename="package://battery_pack/meshes/M6_3_Link.STL" />
-        </geometry>
-      </collision>
-    </link>
-    <joint
-      name="M6_3_Joint"
-      type="fixed">
-      <origin
-        xyz="0.2215 0.204 0.051"
-        rpy="0 0 0" />
-      <parent
-        link="battery_pack_base_link" />
-      <child
-        link="M6_3_Link" />
-      <axis
-        xyz="0 0 1" />
-    </joint>
-    <link
-      name="M8_1_Link">
-      <inertial>
-        <origin
-          xyz="-2.382E-08 -1.0658E-07 -0.014181"
-          rpy="0 0 0" />
-        <mass
-          value="0.0021494" />
-        <inertia
-          ixx="2.2689E-07"
-          ixy="3.8573E-12"
-          ixz="-1.3221E-11"
-          iyy="2.2689E-07"
-          iyz="9.8346E-11"
-          izz="2.5923E-08" />
-      </inertial>
-      <visual>
-        <origin
-          xyz="0 0 0"
-          rpy="0 0 0" />
-        <geometry>
-          <mesh
-            filename="package://battery_pack/meshes/M8_1_Link.STL" />
-        </geometry>
-        <material
-          name="">
-          <color
-            rgba="1 1 1 1" />
-        </material>
-      </visual>
-      <collision>
-        <origin
-          xyz="0 0 0"
-          rpy="0 0 0" />
-        <geometry>
-          <mesh
-            filename="package://battery_pack/meshes/M8_1_Link.STL" />
-        </geometry>
-      </collision>
-    </link>
-    <joint
-      name="M8_1_Joint"
-      type="fixed">
-      <origin
-        xyz="0.2215 0.104 0.051"
-        rpy="0 0 0" />
-      <parent
-        link="battery_pack_base_link" />
-      <child
-        link="M8_1_Link" />
-      <axis
-        xyz="0 0 1" />
-    </joint>
-    <link
-      name="M8_2_Link">
-      <inertial>
-        <origin
-          xyz="-1.0237E-07 3.8028E-08 -0.014181"
-          rpy="0 0 0" />
-        <mass
-          value="0.0021494" />
-        <inertia
-          ixx="2.2689E-07"
-          ixy="-3.7109E-12"
-          ixz="9.9231E-11"
-          iyy="2.2689E-07"
-          iyz="-2.1345E-13"
-          izz="2.5923E-08" />
-      </inertial>
-      <visual>
-        <origin
-          xyz="0 0 0"
-          rpy="0 0 0" />
-        <geometry>
-          <mesh
-            filename="package://battery_pack/meshes/M8_2_Link.STL" />
-        </geometry>
-        <material
-          name="">
-          <color
-            rgba="1 1 1 1" />
-        </material>
-      </visual>
-      <collision>
-        <origin
-          xyz="0 0 0"
-          rpy="0 0 0" />
-        <geometry>
-          <mesh
-            filename="package://battery_pack/meshes/M8_2_Link.STL" />
-        </geometry>
-      </collision>
-    </link>
-    <joint
-      name="M8_2_Joint"
-      type="fixed">
-      <origin
-        xyz="0.2215 0.004 0.051"
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