Commit message: add camera plugin

File: rokae/src/gazebo_link_attacher_ws/src/battery_pack/urdf/battery_pack.urdf (robot description, URDF)
Before this commit: robot battery_pack, 11 links, 10 joints
Links:
- removed link M10_1_Link
- removed link M10_2_Link
- removed link M10_3_Link
- removed link M6_1_Link
- removed link M6_2_Link
- removed link M6_3_Link
- removed link M8_1_Link
- removed link M8_2_Link
- removed link M8_3_Link
- removed link sleeve_plate_Link
- added link M10_bolt_1_link, mass 0.003184; collision mesh filename=package://battery_pack/meshes/M10_bolt_1_link.STL; visual mesh filename=package://battery_pack/meshes/M10_bolt_1_link.STL
- added link M10_bolt_2_link, mass 0.003184; collision mesh filename=package://battery_pack/meshes/M10_bolt_2_link.STL; visual mesh filename=package://battery_pack/meshes/M10_bolt_2_link.STL
- added link M10_bolt_3_link, mass 0.003184; collision mesh filename=package://battery_pack/meshes/M10_bolt_3_link.STL; visual mesh filename=package://battery_pack/meshes/M10_bolt_3_link.STL
- added link M10_gasket_1_link, mass 0.00014002; collision mesh filename=package://battery_pack/meshes/M10_gasket_1_link.STL; visual mesh filename=package://battery_pack/meshes/M10_gasket_1_link.STL
- added link M10_gasket_2_link, mass 0.00014002; collision mesh filename=package://battery_pack/meshes/M10_gasket_2_link.STL; visual mesh filename=package://battery_pack/meshes/M10_gasket_2_link.STL
- added link M10_gasket_3_link, mass 0.00014002; collision mesh filename=package://battery_pack/meshes/M10_gasket_3_link.STL; visual mesh filename=package://battery_pack/meshes/M10_gasket_3_link.STL
- added link M6_bolt_1_link, mass 0.0013212; collision mesh filename=package://battery_pack/meshes/M6_bolt_1_link.STL; visual mesh filename=package://battery_pack/meshes/M6_bolt_1_link.STL
- added link M6_bolt_2_link, mass 0.0013212; collision mesh filename=package://battery_pack/meshes/M6_bolt_2_link.STL; visual mesh filename=package://battery_pack/meshes/M6_bolt_2_link.STL
- added link M6_bolt_3_link, mass 0.0013212; collision mesh filename=package://battery_pack/meshes/M6_bolt_3_link.STL; visual mesh filename=package://battery_pack/meshes/M6_bolt_3_link.STL
- added link M6_gasket_1_link, mass 9.9286E-05; collision mesh filename=package://battery_pack/meshes/M6_gasket_1_link.STL; visual mesh filename=package://battery_pack/meshes/M6_gasket_1_link.STL
- added link M6_gasket_2_link, mass 9.9286E-05; collision mesh filename=package://battery_pack/meshes/M6_gasket_2_link.STL; visual mesh filename=package://battery_pack/meshes/M6_gasket_2_link.STL
- added link M6_gasket_3_link, mass 9.9286E-05; collision mesh filename=package://battery_pack/meshes/M6_gasket_3_link.STL; visual mesh filename=package://battery_pack/meshes/M6_gasket_3_link.STL
- added link M8_bolt_1_link, mass 0.0021494; collision mesh filename=package://battery_pack/meshes/M8_bolt_1_link.STL; visual mesh filename=package://battery_pack/meshes/M8_bolt_1_link.STL
- added link M8_bolt_2_link, mass 0.0021494; collision mesh filename=package://battery_pack/meshes/M8_bolt_2_link.STL; visual mesh filename=package://battery_pack/meshes/M8_bolt_2_link.STL
- added link M8_bolt_3_link, mass 0.0021494; collision mesh filename=package://battery_pack/meshes/M8_bolt_3_link.STL; visual mesh filename=package://battery_pack/meshes/M8_bolt_3_link.STL
- added link M8_gasket_1_link, mass 0.00011965; collision mesh filename=package://battery_pack/meshes/M8_gasket_1_link.STL; visual mesh filename=package://battery_pack/meshes/M8_gasket_1_link.STL
- added link M8_gasket_2_link, mass 0.00011965; collision mesh filename=package://battery_pack/meshes/M8_gasket_2_link.STL; visual mesh filename=package://battery_pack/meshes/M8_gasket_2_link.STL
- added link M8_gasket_3_link, mass 0.00011965; collision mesh filename=package://battery_pack/meshes/M8_gasket_3_link.STL; visual mesh filename=package://battery_pack/meshes/M8_gasket_3_link.STL
- added link battery_link, mass 0; collision mesh filename=package://battery_pack/meshes/battery_link.STL; visual mesh filename=package://battery_pack/meshes/battery_link.STL
- added link sleeve_plate_link, mass 0.58226; collision mesh filename=package://battery_pack/meshes/sleeve_plate_link.STL; visual mesh filename=package://battery_pack/meshes/sleeve_plate_link.STL
- link battery_pack_base_link: mass 662.17 -> 552
Joints:
- removed joint M10_1_Joint
- removed joint M10_2_Joint
- removed joint M10_3_Joint
- removed joint M6_1_Joint
- removed joint M6_2_Joint
- removed joint M6_3_Joint
- removed joint M8_1_Joint
- removed joint M8_2_Joint
- removed joint M8_3_Joint
- removed joint sleeve_plate_Joint
- added joint M10_bolt_1_joint: type fixed, parent battery_pack_base_link, child M10_bolt_1_link, origin xyz=-0.5215 0.196 0.0485 rpy=0 0 0, axis 0 0 0
- added joint M10_bolt_2_joint: type fixed, parent battery_pack_base_link, child M10_bolt_2_link, origin xyz=-0.5215 0.296 0.0485 rpy=0 0 0, axis 0 0 0
- added joint M10_bolt_3_joint: type fixed, parent battery_pack_base_link, child M10_bolt_3_link, origin xyz=-0.5215 0.396 0.0485 rpy=0 0 0, axis 0 0 0
- added joint M10_gasket_1_joint: type fixed, parent battery_pack_base_link, child M10_gasket_1_link, origin xyz=-0.5215 0.196 0.0485 rpy=0 0 0, axis 0 0 0
- added joint M10_gasket_2_joint: type fixed, parent battery_pack_base_link, child M10_gasket_2_link, origin xyz=-0.5215 0.296 0.0485 rpy=0 0 0, axis 0 0 0
- added joint M10_gasket_3_joint: type fixed, parent battery_pack_base_link, child M10_gasket_3_link, origin xyz=-0.5215 0.396 0.0485 rpy=0 0 0, axis 0 0 0
- added joint M6_bolt_1_joint: type fixed, parent battery_pack_base_link, child M6_bolt_1_link, origin xyz=-0.5215 -0.404 0.0485 rpy=0 0 0, axis 0 0 1
- added joint M6_bolt_2_joint: type fixed, parent battery_pack_base_link, child M6_bolt_2_link, origin xyz=-0.5215 -0.304 0.0485 rpy=0 0 0, axis 0 0 0
- added joint M6_bolt_3_joint: type fixed, parent battery_pack_base_link, child M6_bolt_3_link, origin xyz=-0.5215 -0.204 0.0485 rpy=0 0 0, axis 0 0 0
- added joint M6_gasket_1_joint: type fixed, parent battery_pack_base_link, child M6_gasket_1_link, origin xyz=-0.5215 -0.404 0.0485 rpy=0 0 0, axis 0 0 0
- added joint M6_gasket_2_joint: type fixed, parent battery_pack_base_link, child M6_gasket_2_link, origin xyz=-0.5215 -0.304 0.0485 rpy=0 0 0, axis 0 0 0
- added joint M6_gasket_3_joint: type fixed, parent battery_pack_base_link, child M6_gasket_3_link, origin xyz=-0.5215 -0.204 0.0485 rpy=0 0 0, axis 0 0 0
- added joint M8_bolt_1_joint: type fixed, parent battery_pack_base_link, child M8_bolt_1_link, origin xyz=-0.5215 -0.104 0.0485 rpy=0 0 0, axis 0 0 0
- added joint M8_bolt_2_joint: type fixed, parent battery_pack_base_link, child M8_bolt_2_link, origin xyz=-0.5215 -0.004 0.0485 rpy=0 0 0, axis 0 0 0
- added joint M8_bolt_3_joint: type fixed, parent battery_pack_base_link, child M8_bolt_3_link, origin xyz=-0.5215 0.096 0.0485 rpy=0 0 0, axis 0 0 0
- added joint M8_gasket_1_joint: type fixed, parent battery_pack_base_link, child M8_gasket_1_link, origin xyz=-0.5215 -0.104 0.0485 rpy=0 0 0, axis 0 0 0
- added joint M8_gasket_2_joint: type fixed, parent battery_pack_base_link, child M8_gasket_2_link, origin xyz=-0.5215 -0.004 0.0485 rpy=0 0 0, axis 0 0 0
- added joint M8_gasket_3_joint: type fixed, parent battery_pack_base_link, child M8_gasket_3_link, origin xyz=-0.5215 0.096 0.0485 rpy=0 0 0, axis 0 0 0
- added joint battery_joint: type fixed, parent battery_pack_base_link, child battery_link, origin xyz=-0.504 -0.504 0.035 rpy=0 0 0, axis 0 0 0
- added joint sleeve_plate_joint: type fixed, parent battery_pack_base_link, child sleeve_plate_link, origin xyz=0 0.45 0.065 rpy=0 0 0, axis 0 0 0

File: rokae/src/gazebo_link_attacher_ws/src/fmauch_universal_robot/ur_description/urdf/battery_pack_sleeve/battery_pack.urdf.xacro (robot description, xacro)
@@ -9,45 +9,102 @@
     <inertial>
       <origin
-        xyz="1.011 0.00066689 -0.077539"
-        rpy="0 0 0" />
-      <mass
-        value="662.17" />
-      <inertia
-        ixx="77.302"
-        ixy="0.00076184"
-        ixz="6.3202E-09"
-        iyy="267.99"
-        iyz="1.6099E-09"
-        izz="341.52" />
-    </inertial>
-    <visual>
-      <origin
-        xyz="0 0 0"
-        rpy="0 0 0" />
-      <geometry>
-        <mesh
-          filename="package://battery_pack/meshes/battery_pack_base_link.STL" />
-      </geometry>
-      <material
-        name="">
-        <color
-          rgba="1 1 1 1" />
-      </material>
-    </visual>
-    <collision>
-      <origin
-        xyz="0 0 0"
-        rpy="0 0 0" />
-      <geometry>
-        <mesh
-          filename="package://battery_pack/meshes/battery_pack_base_link.STL" />
-      </geometry>
-    </collision>
-  </link>
-  <link
-    name="M6_1_Link">
-    <inertial>
-      <origin
-        xyz="-1.5781E-08 1.7199E-07 -0.013589"
+        xyz="-0.95 0 -0.1"
+        rpy="0 0 0" />
+      <mass
+        value="552" />
+      <inertia
+        ixx="68.08"
+        ixy="-7.8419E-15"
+        ixz="4.0486E-16"
+        iyy="245.18"
+        iyz="6.6498E-16"
+        izz="309.58" />
+    </inertial>
+    <visual>
+      <origin
+        xyz="0 0 0"
+        rpy="0 0 0" />
+      <geometry>
+        <mesh
+          filename="package://battery_pack/meshes/battery_pack_base_link.dae" />
+      </geometry>
+      <material
+        name="battery">
+        <color
+          rgba="1 1 1 1" />
+        <texture
+          filename="package://battery_pack/textures/battery.png" />
+      </material>
+    </visual>
+    <collision>
+      <origin
+        xyz="0 0 0"
+        rpy="0 0 0" />
+      <geometry>
+        <mesh
+          filename="package://battery_pack/meshes/battery_pack_base_link.dae" />
+      </geometry>
+    </collision>
+  </link>
+  <link
+    name="sleeve_plate_link">
+    <inertial>
+      <origin
+        xyz="0.0005113 -0.00023823 -0.033555"
+        rpy="0 0 0" />
+      <mass
+        value="0.58226" />
+      <inertia
+        ixx="0.00067784"
+        ixy="-7.0925E-08"
+        ixz="-7.5087E-07"
+        iyy="0.00066736"
+        iyz="3.231E-07"
+        izz="0.00093345" />
+    </inertial>
+    <visual>
+      <origin
+        xyz="0 0 0"
+        rpy="0 0 0" />
+      <geometry>
+        <mesh
+          filename="package://battery_pack/meshes/sleeve_plate_link.dae" />
+      </geometry>
+      <material
+        name="battery">
+        <color
+          rgba="1 1 1 1" />
+        <texture
+          filename="package://battery_pack/textures/battery.png" />
+      </material>
+    </visual>
+    <collision>
+      <origin
+        xyz="0 0 0"
+        rpy="0 0 0" />
+      <geometry>
+        <mesh
+          filename="package://battery_pack/meshes/sleeve_plate_link.dae" />
+      </geometry>
+    </collision>
+  </link>
+  <joint
+    name="sleeve_plate_joint"
+    type="fixed">
+    <origin
+      xyz="0 0.45 0.065"
+      rpy="0 0 0" />
+    <parent
+      link="battery_pack_base_link" />
+    <child
+      link="sleeve_plate_link" />
+    <axis
+      xyz="0 0 0" />
+  </joint>
+  <link
+    name="M6_bolt_1_link">
+    <inertial>
+      <origin
+        xyz="-1.0665E-07 -1.3585E-07 -0.011089"
         rpy="0 0 0" />
       <mass
@@ -55,8 +112,8 @@
       <inertia
         ixx="1.3904E-07"
-        ixy="-5.0602E-13"
-        ixz="5.5231E-11"
+        ixy="1.1478E-12"
+        ixz="-2.8329E-11"
         iyy="1.3904E-07"
-        iyz="-1.7203E-11"
+        iyz="5.0437E-11"
         izz="1.0587E-08" />
     </inertial>
@@ -67,305 +124,647 @@
       <geometry>
         <mesh
-          filename="package://battery_pack/meshes/M6_1_Link.STL" />
-      </geometry>
-      <material
-        name="">
-        <color
-          rgba="1 1 1 1" />
-      </material>
-    </visual>
-    <collision>
-      <origin
-        xyz="0 0 0"
-        rpy="0 0 0" />
-      <geometry>
-        <mesh
-          filename="package://battery_pack/meshes/M6_1_Link.STL" />
-      </geometry>
-    </collision>
-  </link>
-  <joint
-    name="M6_1_Joint"
-    type="fixed">
-    <origin
-      xyz="0.521499999999999 0.404 0.051"
-      rpy="0 0 0" />
-    <parent
-      link="battery_pack_base_link" />
-    <child
-      link="M6_1_Link" />
+          filename="package://battery_pack/meshes/M6_bolt_1_link.dae" />
+      </geometry>
+      <material
+        name="bolt">
+        <color
+          rgba="1 1 1 1" />
+        <texture
+          filename="package://battery_pack/textures/bolt_color.jpg" />
+      </material>
+    </visual>
+    <collision>
+      <origin
+        xyz="0 0 0"
+        rpy="0 0 0" />
+      <geometry>
+        <mesh
+          filename="package://battery_pack/meshes/M6_bolt_1_link.dae" />
+      </geometry>
+    </collision>
+  </link>
+  <joint
+    name="M6_bolt_1_joint"
+    type="fixed">
+    <origin
+      xyz="-0.5215 -0.404 0.0485"
+      rpy="0 0 0" />
+    <parent
+      link="battery_pack_base_link" />
+    <child
+      link="M6_bolt_1_link" />
     <axis
       xyz="0 0 1" />
   </joint>
   <link
-    name="M6_2_Link">
-    <inertial>
-      <origin
-        xyz="-1.69178282917459E-07 -3.47719712190386E-08 -0.0135893488314754"
-        rpy="0 0 0" />
-      <mass
-        value="0.0013211670322828" />
-      <inertia
-        ixx="1.39039904452008E-07"
-        ixy="7.53479092438269E-13"
-        ixz="1.09674715667674E-11"
-        iyy="1.39037829163727E-07"
-        iyz="5.67986038374194E-11"
-        izz="1.05870312742737E-08" />
-    </inertial>
-    <visual>
-      <origin
-        xyz="0 0 0"
-        rpy="0 0 0" />
-      <geometry>
-        <mesh
-          filename="package://battery_pack/meshes/M6_2_Link.STL" />
-      </geometry>
-      <material
-        name="">
-        <color
-          rgba="1 1 1 1" />
-      </material>
-    </visual>
-    <collision>
-      <origin
-        xyz="0 0 0"
-        rpy="0 0 0" />
-      <geometry>
-        <mesh
-          filename="package://battery_pack/meshes/M6_2_Link.STL" />
-      </geometry>
-    </collision>
-  </link>
-  <joint
-    name="M6_2_Joint"
-    type="fixed">
-    <origin
-      xyz="0.521499999999999 0.304000000000001 0.051"
-      rpy="0 0 0" />
-    <parent
-      link="battery_pack_base_link" />
-    <child
-      link="M6_2_Link" />
-    <axis
-      xyz="0 0 1" />
-  </joint>
-  <link
-    name="M6_3_Link">
-    <inertial>
-      <origin
-        xyz="-8.60276639161328E-09 -1.7250035883043E-07 -0.0135893488314759"
-        rpy="0 0 0" />
-      <mass
-        value="0.00132116703228283" />
-      <inertia
-        ixx="1.39037594136452E-07"
-        ixy="-1.57300860848985E-13"
-        ixz="-5.22565946292113E-11"
-        iyy="1.39040139479292E-07"
-        iyz="2.4811593020993E-11"
-        izz="1.0587031274274E-08" />
-    </inertial>
-    <visual>
-      <origin
-        xyz="0 0 0"
-        rpy="0 0 0" />
-      <geometry>
-        <mesh
-          filename="package://battery_pack/meshes/M6_3_Link.STL" />
-      </geometry>
-      <material
-        name="">
-        <color
-          rgba="1 1 1 1" />
-      </material>
-    </visual>
-    <collision>
-      <origin
-        xyz="0 0 0"
-        rpy="0 0 0" />
-      <geometry>
-        <mesh
-          filename="package://battery_pack/meshes/M6_3_Link.STL" />
-      </geometry>
-    </collision>
-  </link>
-  <joint
-    name="M6_3_Joint"
-    type="fixed">
-    <origin
-      xyz="0.521499999999999 0.204000000000001 0.051"
-      rpy="0 0 0" />
-    <parent
-      link="battery_pack_base_link" />
-    <child
-      link="M6_3_Link" />
-    <axis
-      xyz="0 0 1" />
-  </joint>
-  <link
-    name="M8_1_Link">
-    <inertial>
-      <origin
-        xyz="-2.38202364499784E-08 -1.06578474601271E-07 -0.0141810682031523"
-        rpy="0 0 0" />
-      <mass
-        value="0.00214941637065255" />
-      <inertia
-        ixx="2.26889617708073E-07"
-        ixy="3.85731537612252E-12"
-        ixz="-1.32208549983177E-11"
-        iyy="2.26889580273997E-07"
-        iyz="9.83462091995749E-11"
-        izz="2.59232568951157E-08" />
-    </inertial>
-    <visual>
-      <origin
-        xyz="0 0 0"
-        rpy="0 0 0" />
-      <geometry>
-        <mesh
-          filename="package://battery_pack/meshes/M8_1_Link.STL" />
-      </geometry>
-      <material
-        name="">
-        <color
-          rgba="1 1 1 1" />
-      </material>
-    </visual>
-    <collision>
-      <origin
-        xyz="0 0 0"
-        rpy="0 0 0" />
-      <geometry>
-        <mesh
-          filename="package://battery_pack/meshes/M8_1_Link.STL" />
-      </geometry>
-    </collision>
-  </link>
-  <joint
-    name="M8_1_Joint"
-    type="fixed">
-    <origin
-      xyz="0.521499999999999 0.104000000000001 0.051"
-      rpy="0 0 0" />
-    <parent
-      link="battery_pack_base_link" />
-    <child
-      link="M8_1_Link" />
-    <axis
-      xyz="0 0 1" />
-  </joint>
-  <link
-    name="M8_2_Link">
-    <inertial>
-      <origin
-        xyz="-1.02373083312596E-07 3.80279728817712E-08 -0.014181068203152"
-        rpy="0 0 0" />
-      <mass
-        value="0.00214941637065243" />
-      <inertia
-        ixx="2.26888546281706E-07"
-        ixy="-3.71093456176309E-12"
-        ixz="9.92306520596295E-11"
-        iyy="2.26890651700353E-07"
-        iyz="-2.1345480205816E-13"
-        izz="2.59232568951147E-08" />
-    </inertial>
-    <visual>
-      <origin
-        xyz="0 0 0"
-        rpy="0 0 0" />
-      <geometry>
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
File: rokae/src/gazebo_link_attacher_ws/src/fmauch_universal_robot/ur_description/urdf/battery_pack_sleeve/endeffector.urdf.xacro (robot description, xacro)
@@ -104,3 +104,9 @@
         <child link="endeffector_base_link"/>
       </joint>
+  <link name="camera_gz_Link"/>
+  <joint name="camera_gz_joint" type="fixed">
+      <origin xyz="0 0 0" rpy="0 ${-pi/2.0} ${pi/2.0}" />
+      <parent link="camera_Link" />
+      <child link="camera_gz_Link" />
+  </joint>
 </robot>

File: rokae/src/gazebo_link_attacher_ws/src/fmauch_universal_robot/ur_description/urdf/inc/ur_macro.xacro (robot description, xacro)
@@ -319,4 +319,4 @@
   <xacro:include filename="$(find ur_description)/urdf/battery_pack_sleeve/battery_pack.urdf.xacro" />
   <xacro:include filename="$(find ur_description)/urdf/battery_pack_sleeve/endeffector.urdf.xacro" />
-  <xacro:include filename="$(find ur_description)/urdf/sensors/sensor_kinect.urdf.xacro" />
+  <xacro:include filename="$(find ur_description)/urdf/sensors/_d435.gazebo.xacro" />
 </robot>
