Commit message: gazebo complete the camera message publish to ROS

File: rokae/src/gazebo_link_attacher_ws/src/fmauch_universal_robot/ur_description/urdf/inc/ur_macro.xacro (robot description, xacro)
@@ -319,4 +319,4 @@
   <xacro:include filename="$(find ur_description)/urdf/battery_pack_sleeve/battery_pack.urdf.xacro" />
   <xacro:include filename="$(find ur_description)/urdf/battery_pack_sleeve/endeffector.urdf.xacro" />
-  <xacro:include filename="$(find ur_description)/urdf/sensors/_d435.gazebo.xacro" />
+  <xacro:include filename="$(find ur_description)/urdf/sensors/_d435.urdf.xacro" />
 </robot>

File: rokae/src/gazebo_link_attacher_ws/src/fmauch_universal_robot/ur_description/urdf/sensors/_d435.gazebo.xacro (robot description, xacro)
@@ -6,5 +6,5 @@
 -->
 <robot xmlns:xacro="http://ros.org/wiki/xacro">
-    <xacro:property name="deg_to_rad" value="0.01745329251994329577" />
+<xacro:property name="deg_to_rad" value="0.01745329251994329577" />
     <gazebo reference="camera_gz_Link">
       <self_collide>0</self_collide>
@@ -109,5 +109,5 @@
       </sensor>
     </gazebo>
-    <gazebo>
+    <!-- <gazebo>
       <plugin name="camera" filename="librealsense_gazebo_plugin.so">
         <prefix>camera</prefix>
@@ -134,4 +134,4 @@
         <pointCloudCutoffMax>9.0</pointCloudCutoffMax>
       </plugin>
-    </gazebo>
+    </gazebo>  -->
 </robot>
