Commit message: change the ur_end_effector model

File: rokae/src/ur_real_robot/socket_describe/urdf/socket_jacket.xacro (robot description, xacro)
@@ -3,84 +3,156 @@
      Commit Version: 1.5.1-0-g916b5db  Build Version: 1.5.7152.31018
      For more information, please see http://wiki.ros.org/sw_urdf_exporter -->
-<robot name="socket_describe"
-  xmlns:xacro="http://www.ros.org/wiki/xacro">
-  <link name="pneumatic_base_link">
+<robot
+  name="socket_describe">
+  <link
+    name="pneumatic_base_link">
     <inertial>
-      <origin xyz="2.3901E-06 -0.031661 -0.082455" rpy="0 0 0" />
-      <mass value="0.63254" />
-      <inertia ixx="0.0016249" ixy="-2.4777E-08" ixz="-8.1418E-08" iyy="0.00061245" iyz="4.3555E-05" izz="0.0012505" />
+      <origin
+        xyz="0.0099146 -5.4634E-05 0.088854"
+        rpy="0 0 0" />
+      <mass
+        value="0.64615" />
+      <inertia
+        ixx="0.00070554"
+        ixy="-1.6495E-06"
+        ixz="2.4231E-05"
+        iyy="0.0016576"
+        iyz="1.9116E-06"
+        izz="0.0011985" />
     </inertial>
     <visual>
-      <origin xyz="0 0 0" rpy="0 0 0" />
+      <origin
+        xyz="0 0 0"
+        rpy="0 0 0" />
       <geometry>
-        <mesh filename="package://socket_describe/meshes/pneumatic_base_link.STL" />
+        <mesh
+          filename="package://socket_describe/meshes/pneumatic_base_link.STL" />
       </geometry>
-      <material name="">
-        <color rgba="1 1 1 1" />
+      <material
+        name="">
+        <color
+          rgba="0.53 0.81 0.92 1" />
       </material>
     </visual>
     <collision>
-      <origin xyz="0 0 0" rpy="0 0 0" />
+      <origin
+        xyz="0 0 0"
+        rpy="0 0 0" />
       <geometry>
-        <mesh filename="package://socket_describe/meshes/pneumatic_base_link.STL" />
+        <mesh
+          filename="package://socket_describe/meshes/pneumatic_base_link.STL" />
       </geometry>
     </collision>
   </link>
-  <link name="sleeve_Link">
+  <link
+    name="camera_Link">
     <inertial>
-      <origin xyz="-6.2102E-10 2.2153E-09 -0.27064" rpy="0 0 0" />
-      <mass value="0.059247" />
-      <inertia ixx="0.00026061" ixy="-2.3096E-13" ixz="-1.6484E-12" iyy="0.00026061" iyz="1.0567E-11" izz="2.6182E-06" />
+      <origin
+        xyz="0.013488 7.0938E-05 -0.013332"
+        rpy="0 0 0" />
+      <mass
+        value="0.071592" />
+      <inertia
+        ixx="2.0232E-05"
+        ixy="-4.6475E-08"
+        ixz="5.1114E-10"
+        iyy="1.9381E-05"
+        iyz="-4.5469E-09"
+        izz="3.1685E-05" />
     </inertial>
     <visual>
-      <origin xyz="0 0 0" rpy="0 0 0" />
+      <origin
+        xyz="0 0 0"
+        rpy="0 0 0" />
       <geometry>
-        <mesh filename="package://socket_describe/meshes/sleeve_Link.STL" />
+        <mesh
+          filename="package://socket_describe/meshes/camera_Link.STL" />
       </geometry>
-      <material name="">
-        <color rgba="1 1 1 1" />
+      <material
+        name="">
+        <color
+          rgba="0.7 0.7 0.7 1.0" />
       </material>
     </visual>
     <collision>
-      <origin xyz="0 0 0" rpy="0 0 0" />
+      <origin
+        xyz="0 0 0"
+        rpy="0 0 0" />
       <geometry>
-        <mesh filename="package://socket_describe/meshes/sleeve_Link.STL" />
+        <mesh
+          filename="package://socket_describe/meshes/camera_Link.STL" />
       </geometry>
     </collision>
   </link>
-  <joint name="sleeve_joint" type="continuous">
-    <origin xyz="0 0 0" rpy="0 0 0" />
-    <parent link="pneumatic_base_link" />
-    <child link="sleeve_Link" />
-    <axis xyz="0 0 -1" />
+  <joint
+    name="camera_Joint"
+    type="fixed">
+    <origin
+      xyz="-0.18055 -0.00090604 0.071047"
+      rpy="0.016843 0.10474 0.0017763" />
+    <parent
+      link="pneumatic_base_link" />
+    <child
+      link="camera_Link" />
+    <axis
+      xyz="0 0 0" />
   </joint>
-  <link name="camera_Link">
+  <link
+    name="sleeve_Link">
     <inertial>
-      <origin xyz="-0.0040157 2.614E-05 -0.075782" rpy="0 0 0" />
-      <mass value="0.12805" />
-      <inertia ixx="0.00010423" ixy="-4.9755E-10" ixz="6.6151E-07" iyy="9.2528E-05" iyz="-4.8206E-08" izz="3.1847E-05" />
+      <origin
+        xyz="-3.2497E-09 2.024E-09 -0.16147"
+        rpy="0 0 0" />
+      <mass
+        value="0.059949" />
+      <inertia
+        ixx="0.00026672"
+        ixy="3.9947E-13"
+        ixz="1.5755E-11"
+        iyy="0.00026672"
+        iyz="-9.4277E-12"
+        izz="2.6369E-06" />
     </inertial>
     <visual>
-      <origin xyz="0 0 0" rpy="0 0 0" />
+      <origin
+        xyz="0 0 0"
+        rpy="0 0 0" />
       <geometry>
-        <mesh filename="package://socket_describe/meshes/camera_Link.STL" />
+        <mesh
+          filename="package://socket_describe/meshes/sleeve_Link.STL" />
       </geometry>
-      <material name="">
-        <color rgba="1 1 1 1" />
+      <material
+        name="">
+        <color
+          rgba="0.7 0.7 0.7 1.0" />
       </material>
     </visual>
     <collision>
-      <origin xyz="0 0 0" rpy="0 0 0" />
+      <origin
+        xyz="0 0 0"
+        rpy="0 0 0" />
       <geometry>
-        <mesh filename="package://socket_describe/meshes/camera_Link.STL" />
+        <mesh
+          filename="package://socket_describe/meshes/sleeve_Link.STL" />
       </geometry>
     </collision>
   </link>
-  <joint name="camera_joint" type="prismatic">
-    <origin xyz="0 0.055 -0.07478" rpy="1.5708 -1.5708 0" />
-    <parent link="pneumatic_base_link" />
-    <child link="camera_Link" />
-    <axis xyz="1 0 0" />
-    <limit lower="0" upper="0" effort="0" velocity="0" />
+  <joint
+    name="effect_Joint"
+    type="continuous">
+    <origin
+      xyz="0 0 0.53934"
+      rpy="0 0 0" />
+    <parent
+      link="pneumatic_base_link" />
+    <child
+      link="sleeve_Link" />
+    <axis
+      xyz="0 0 0" />
+    <limit
+      lower="0"
+      upper="0"
+      effort="0"
+      velocity="0" />
   </joint>
 </robot>
