Commit message: model update

File: rokae/src/ur_real_robot/fmauch_universal_robot/ur_description/urdf/inc/ur_macro.xacro (robot description, xacro)
@@ -64,4 +64,21 @@
     <xacro:ur_arm_transmission prefix="${prefix}" hw_interface="${transmission_hw_interface}" />
     <!-- links: main serial chain -->
+    <link name="ground_plane_box">
+      <visual>
+        <origin xyz="0 0 0" rpy="0 0 0"/>
+        <geometry>
+          <box size="3 3 0.05"/>
+        </geometry>
+        <material name="Grey">
+          <color rgba="0.7 0.7 0.7 1.0"/>
+        </material>
+      </visual>
+      <collision>
+        <origin xyz="0 0 0" rpy="0 0 0"/>
+        <geometry>
+          <box size="3 3 0.05"/>
+        </geometry>
+      </collision>
+    </link>
     <link name="${prefix}base_link"/>
     <link name="${prefix}base_link_inertia">
@@ -207,4 +224,9 @@
     </link>
     <!-- joints: main serial chain -->
+    <joint name="ground_plane_box" type="fixed">
+      <parent link="base" />
+      <child link="ground_plane_box" />
+      <origin xyz="0 0 0" rpy="0 0 0" />
+    </joint>
     <joint name="${prefix}base_link-base_link_inertia" type="fixed">
       <parent link="${prefix}base_link" />

File: rokae/src/ur_real_robot/ur_socket_describe/urdf/ur_socket_complex.xacro (robot description, xacro)
@@ -5,5 +5,5 @@
   <xacro:include filename="$(find socket_describe)/urdf/socket_jacket.xacro" />
   <joint name="ur_socket_joint" type="fixed">
-    <origin xyz="0 0 -0.007" rpy="0  ${pi}   ${pi/2}  " />
+    <origin xyz="0 0 -0.007" rpy="0  0   0  " />
     <parent link="tool0"/>
     <child link="pneumatic_base_link"/>
