Commit message: fix bug of urdf

File: rokae/src/ur_real_robot/ur_socket_describe/urdf/ur_socket_complex.xacro (robot description, xacro)
@@ -5,5 +5,5 @@
   <xacro:include filename="$(find socket_describe)/urdf/socket_jacket.xacro" />
   <joint name="ur_socket_joint" type="fixed">
-    <origin xyz="0 0 -0.007" rpy="0  ${pi}   ${pi/2}  " />
+    <origin xyz="0 0 -0.007" rpy="0  0  0 " />
     <parent link="tool0"/>
     <child link="pneumatic_base_link"/>

Commit message: model updated

File: rokae/src/ur_real_robot/ur_socket_describe/urdf/ur_socket_complex.xacro (robot description, xacro)
@@ -5,5 +5,5 @@
   <xacro:include filename="$(find socket_describe)/urdf/socket_jacket.xacro" />
   <joint name="ur_socket_joint" type="fixed">
-    <origin xyz="0 0 -0.007" rpy="0  0  0 " />
+    <origin xyz="0 0 -0.007" rpy="0  0   0  " />
     <parent link="tool0"/>
     <child link="pneumatic_base_link"/>

Commit message: model updated 0721

File: rokae/src/ur_real_robot/ur_socket_describe/urdf/ur_socket_complex.xacro (robot description, xacro)
@@ -3,7 +3,7 @@
   <xacro:include filename="$(find ur_description)/urdf/inc/ur10e_macro.xacro"/>
   <xacro:ur10e_robot prefix="" />
-  <xacro:include filename="$(find socket_describe)/urdf/socket_jacket.xacro" />
+  <xacro:include filename="$(find end_effector)/urdf/end_effector.urdf" />
   <joint name="ur_socket_joint" type="fixed">
-    <origin xyz="0 0 -0.007" rpy="0  0   0  " />
+    <origin xyz="0 0 0" rpy="0  -1.57   0  " />
     <parent link="tool0"/>
     <child link="pneumatic_base_link"/>
