Commit message: roslaunch ur_gazebo ur10e_bringup.launch

File: gazebo_link_attacher_ws/src/fmauch_universal_robot/ur_description/urdf/battery_pack_sleeve/battery_pack.urdf.xacro (robot description, xacro)
@@ -4,19 +4,19 @@
      For more information, please see http://wiki.ros.org/sw_urdf_exporter -->
 <robot
-  name="battery_pack">
+  name="battery_pack_3">
   <link
     name="battery_pack_base_link">
     <inertial>
       <origin
-        xyz="-0.95 0 -0.1"
+        xyz="-0.95 0 -0.0999999999999996"
         rpy="0 0 0" />
       <mass
         value="552" />
       <inertia
-        ixx="68.08"
-        ixy="-7.8419E-15"
-        ixz="4.0486E-16"
+        ixx="68.0799999999999"
+        ixy="-7.84187529726902E-15"
+        ixz="-1.07543603652023E-15"
         iyy="245.18"
-        iyz="6.6498E-16"
+        iyz="1.32995466491555E-16"
         izz="309.58" />
     </inertial>
@@ -27,5 +27,5 @@
       <geometry>
         <mesh
-          filename="package://battery_pack/meshes/battery_pack_base_link.dae" />
+          filename="package://battery_pack_3/meshes/battery_pack_base_link.dae" />
       </geometry>
       <material
@@ -33,41 +33,410 @@
         <color
           rgba="1 1 1 1" />
-        <texture
-          filename="package://battery_pack/textures/battery.png" />
-      </material>
-    </visual>
-    <collision>
-      <origin
-        xyz="0 0 0"
-        rpy="0 0 0" />
-      <geometry>
-        <mesh
-          filename="package://battery_pack/meshes/battery_pack_base_link.dae" />
-      </geometry>
-    </collision>
-  </link>
+      </material>
+    </visual>
+    <collision>
+      <origin
+        xyz="0 0 0"
+        rpy="0 0 0" />
+      <geometry>
+        <mesh
+          filename="package://battery_pack_3/meshes/battery_pack_base_link.dae" />
+      </geometry>
+    </collision>
+  </link>
+  <link
+    name="M6_gasket_1_link">
+    <inertial>
+      <origin
+        xyz="-5.55111512312578E-17 1.11022302462516E-16 -0.000499999999999723"
+        rpy="0 0 0" />
+      <mass
+        value="8.82772243861937E-05" />
+      <inertia
+        ixx="1.24959661693432E-09"
+        ixy="-2.58493941422821E-26"
+        ixz="7.02201084753254E-41"
+        iyy="1.24959661693432E-09"
+        iyz="-1.65030964290011E-40"
+        izz="2.48456062424061E-09" />
+    </inertial>
+    <visual>
+      <origin
+        xyz="0 0 0"
+        rpy="0 0 0" />
+      <geometry>
+        <mesh
+          filename="package://battery_pack_3/meshes/M6_gasket_1_link.dae" />
+      </geometry>
+      <material
+        name="bolt">
+        <color
+          rgba="1 1 1 1" />
+      </material>
+    </visual>
+    <collision>
+      <origin
+        xyz="0 0 0"
+        rpy="0 0 0" />
+      <geometry>
+        <mesh
+          filename="package://battery_pack_3/meshes/M6_gasket_1_link.dae" />
+      </geometry>
+    </collision>
+  </link>
+  <joint
+    name="M6_gasket_1_joint"
+    type="fixed">
+    <origin
+      xyz="-0.5215 -0.404 0.0525"
+      rpy="3.1416 0 -2.7485" />
+    <parent
+      link="battery_pack_base_link" />
+    <child
+      link="M6_gasket_1_link" />
+    <axis
+      xyz="0 0 0" />
+  </joint>
+  <link
+    name="M6_gasket_2_link">
+    <inertial>
+      <origin
+        xyz="0 0 -0.000499999999999723"
+        rpy="0 0 0" />
+      <mass
+        value="8.82772243861937E-05" />
+      <inertia
+        ixx="1.24959661693432E-09"
+        ixy="-1.29246970711411E-25"
+        ixz="1.50034156156908E-42"
+        iyy="1.24959661693432E-09"
+        iyz="6.8771134273246E-43"
+        izz="2.48456062424061E-09" />
+    </inertial>
+    <visual>
+      <origin
+        xyz="0 0 0"
+        rpy="0 0 0" />
+      <geometry>
+        <mesh
+          filename="package://battery_pack_3/meshes/M6_gasket_2_link.dae" />
+      </geometry>
+      <material
+        name="bolt">
+        <color
+          rgba="1 1 1 1" />
+      </material>
+    </visual>
+    <collision>
+      <origin
+        xyz="0 0 0"
+        rpy="0 0 0" />
+      <geometry>
+        <mesh
+          filename="package://battery_pack_3/meshes/M6_gasket_2_link.dae" />
+      </geometry>
+    </collision>
+  </link>
+  <joint
+    name="M6_gasket_2_joint"
+    type="fixed">
+    <origin
+      xyz="-0.5215 -0.304 0.0525"
+      rpy="3.1416 0 -2.7485" />
+    <parent
+      link="battery_pack_base_link" />
+    <child
+      link="M6_gasket_2_link" />
+    <axis
+      xyz="0 0 0" />
+  </joint>
+  <link
+    name="M8_gasket_1_link">
+    <inertial>
+      <origin
+        xyz="0 0 -0.000499999999999945"
+        rpy="0 0 0" />
+      <mass
+        value="0.00010550204865667" />
+      <inertia
+        ixx="2.08686937076162E-09"
+        ixy="5.16987882845642E-26"
+        ixz="1.7437435717737E-42"
+        iyy="2.08686937076162E-09"
+        iyz="2.84281637081175E-43"
+        izz="4.15625098855316E-09" />
+    </inertial>
+    <visual>
+      <origin
+        xyz="0 0 0"
+        rpy="0 0 0" />
+      <geometry>
+        <mesh
+          filename="package://battery_pack_3/meshes/M8_gasket_1_link.dae" />
+      </geometry>
+      <material
+        name="bolt">
+        <color
+          rgba="1 1 1 1" />
+      </material>
+    </visual>
+    <collision>
+      <origin
+        xyz="0 0 0"
+        rpy="0 0 0" />
+      <geometry>
+        <mesh
+          filename="package://battery_pack_3/meshes/M8_gasket_1_link.dae" />
+      </geometry>
+    </collision>
+  </link>
+  <joint
+    name="M8_gasket_1_joint"
+    type="fixed">
+    <origin
+      xyz="-0.5215 -0.104 0.0525"
+      rpy="3.1416 0 -2.7485" />
+    <parent
+      link="battery_pack_base_link" />
+    <child
+      link="M8_gasket_1_link" />
+    <axis
+      xyz="0 0 0" />
+  </joint>
+  <link
+    name="M8_gasket_2_link">
+    <inertial>
+      <origin
+        xyz="0 0 -0.000499999999999945"
+        rpy="0 0 0" />
+      <mass
+        value="0.00010550204865667" />
+      <inertia
+        ixx="2.08686937076162E-09"
+        ixy="5.16987882845642E-26"
+        ixz="1.7437435717737E-42"
+        iyy="2.08686937076162E-09"
+        iyz="2.84281637081175E-43"
+        izz="4.15625098855316E-09" />
+    </inertial>
+    <visual>
+      <origin
+        xyz="0 0 0"
+        rpy="0 0 0" />
+      <geometry>
+        <mesh
+          filename="package://battery_pack_3/meshes/M8_gasket_2_link.dae" />
+      </geometry>
+      <material
+        name="bolt">
+        <color
+          rgba="1 1 1 1" />
+      </material>
+    </visual>
+    <collision>
+      <origin
+        xyz="0 0 0"
+        rpy="0 0 0" />
+      <geometry>
+        <mesh
+          filename="package://battery_pack_3/meshes/M8_gasket_2_link.dae" />
+      </geometry>
+    </collision>
+  </link>
+  <joint
+    name="M8_gasket_2_joint"
+    type="fixed">
+    <origin
+      xyz="-0.521499999999999 -0.00400000000000011 0.0525"
+      rpy="3.14159265358979 0 -2.74849784316327" />
+    <parent
+      link="battery_pack_base_link" />
+    <child
+      link="M8_gasket_2_link" />
+    <axis
+      xyz="0 0 0" />
+  </joint>
+  <link
+    name="M10_gasket_1_link">
+    <inertial>
+      <origin
+        xyz="2.77555756156289E-17 0 -0.000499999999999723"
+        rpy="0 0 0" />
+      <mass
+        value="0.000122726872927147" />
+      <inertia
+        ixx="3.24064827055894E-09"
+        ixy="2.06795153138257E-25"
+        ixz="2.26664384148777E-42"
+        iyy="3.24064827055894E-09"
+        iyz="9.39925665401376E-43"
+        izz="6.46095364480573E-09" />
+    </inertial>
+    <visual>
+      <origin
+        xyz="0 0 0"
+        rpy="0 0 0" />
+      <geometry>
+        <mesh
+          filename="package://battery_pack_3/meshes/M10_gasket_1_link.dae" />
+      </geometry>
+      <material
+        name="bolt">
+        <color
+          rgba="1 1 1 1" />
+      </material>
+    </visual>
+    <collision>
+      <origin
+        xyz="0 0 0"
+        rpy="0 0 0" />
+      <geometry>
+        <mesh
+          filename="package://battery_pack_3/meshes/M10_gasket_1_link.dae" />
+      </geometry>
+    </collision>
+  </link>
+  <joint
+    name="M10_gasket_1_joint"
+    type="fixed">
+    <origin
+      xyz="-0.5215 0.196 0.0525"
+      rpy="3.1416 0 -2.7485" />
+    <parent
+      link="battery_pack_base_link" />
+    <child
+      link="M10_gasket_1_link" />
+    <axis
+      xyz="0 0 0" />
+  </joint>
+  <link
+    name="M10_gasket_2_link">
+    <inertial>
+      <origin
+        xyz="0 0 -0.000499999999999723"
+        rpy="0 0 0" />
+      <mass
+        value="0.000122726872927147" />
+      <inertia
+        ixx="3.24064827055894E-09"
+        ixy="3.10192729707385E-25"
+        ixz="3.07565550259243E-42"
+        iyy="3.24064827055894E-09"
+        iyz="1.27540440712647E-42"
+        izz="6.46095364480573E-09" />
+    </inertial>
+    <visual>
+      <origin
+        xyz="0 0 0"
+        rpy="0 0 0" />
+      <geometry>
+        <mesh
+          filename="package://battery_pack_3/meshes/M10_gasket_2_link.dae" />
+      </geometry>
+      <material
+        name="bolt">
+        <color
+          rgba="1 1 1 1" />
+      </material>
+    </visual>
+    <collision>
+      <origin
+        xyz="0 0 0"
+        rpy="0 0 0" />
+      <geometry>
+        <mesh
+          filename="package://battery_pack_3/meshes/M10_gasket_2_link.dae" />
+      </geometry>
+    </collision>
+  </link>
+  <joint
+    name="M10_gasket_2_joint"
+    type="fixed">
+    <origin
+      xyz="-0.5215 0.296 0.0525"
+      rpy="3.1416 0 -2.7485" />
+    <parent
+      link="battery_pack_base_link" />
+    <child
+      link="M10_gasket_2_link" />
+    <axis
+      xyz="0 0 0" />
+  </joint>
+  <link
+    name="battery_link">
+    <inertial>
+      <origin
+        xyz="-0.812291820172866 0.499989787693561 0"
+        rpy="0 0 0" />
+      <mass
+        value="125.983329440983" />
+      <inertia
+        ixx="10.5619007949744"
+        ixy="0.00102256355122022"
+        ixz="-6.62078457904823E-17"
+        iyy="26.1288590387794"
+        iyz="-7.60212567544936E-17"
+        izz="36.5573338075084" />
+    </inertial>
+    <visual>
+      <origin
+        xyz="0 0 0"
+        rpy="0 0 0" />
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
File: gazebo_link_attacher_ws/src/fmauch_universal_robot/ur_description/urdf/sensors/_d435.urdf.xacro (robot description, xacro)
@@ -12,17 +12,24 @@
      publishing TF values with actual calibrated camera extrinsic values -->
     <xacro:property name="d435_cam_depth_to_left_ir_offset" value="0.0"/>
-    <xacro:property name="d435_cam_depth_to_right_ir_offset" value="-0.050"/>
-    <xacro:property name="d435_cam_depth_to_color_offset" value="0.015"/>
+    <xacro:property name="d435_cam_depth_to_right_ir_offset" value="0.0"/>
+    <!-- -0.050 -->
+    <xacro:property name="d435_cam_depth_to_color_offset" value="0.0"/>
+    <!-- 0.015 -->
     <!-- The following values model the aluminum peripherial case for the
     D435 camera, with the camera joint represented by the actual
     peripherial camera tripod mount -->
-    <xacro:property name="d435_cam_width" value="0.090"/>
-    <xacro:property name="d435_cam_height" value="0.025"/>
-    <xacro:property name="d435_cam_depth" value="0.02505"/>
-    <xacro:property name="d435_cam_mount_from_center_offset" value="0.0149"/>
+    <xacro:property name="d435_cam_width" value="0.0"/>
+    <!-- 0.090 -->
+    <xacro:property name="d435_cam_height" value="0.0"/>
+    <!-- 0.025 -->
+    <xacro:property name="d435_cam_depth" value="0.0"/>
+    <!-- 0.02505 -->
+    <xacro:property name="d435_cam_mount_from_center_offset" value="0.0"/>
+    <!-- 0.0149 -->
     <!-- The following offset is relative the the physical D435 camera peripherial
     camera tripod mount -->
     <xacro:property name="d435_cam_depth_px" value="${d435_cam_mount_from_center_offset}"/>
-    <xacro:property name="d435_cam_depth_py" value="0.0175"/>
+    <xacro:property name="d435_cam_depth_py" value="0.0"/>
+    <!-- 0.0175 -->
     <xacro:property name="d435_cam_depth_pz" value="${d435_cam_height/2}"/>
     <gazebo reference="camera_gz_Link">
